File: PCB/hackboard.kicad_sch (KiCad schematic)
At the start: 175 parts

Commit message: Updated symbols and routing
Parts:
- D_0, D_1, D_10, D_11, D_12, D_13, D_14, D_15, D_16, D_17, D_18, D_19, D_2, D_20, D_21, D_22, D_23, D_24, D_25, D_26, D_27, D_28, D_29, D_3, D_30, D_31, D_32, D_33, D_34, D_35, D_36, D_37, D_38, D_39, D_4, D_40, D_41, D_42, D_43, D_44, D_45, D_46, D_47, D_48, D_49, D_5, D_50, D_51, D_52, D_53, D_54, D_55, D_56, D_57, D_58, D_59, D_6, D_60, D_61, D_62, D_63, D_64, D_65, D_66, D_67, D_68, D_69, D_7, D_70, D_71, D_72, D_73, D_74, D_75, D_76, D_77, D_78, D_79, D_8, D_80, D_81, D_82, D_83, D_84, D_85, D_86, D_9: value D -> 1N4148; symbol Device:D_Small -> Diode:1N4148
- K_0, K_1, K_10, K_11, K_12, K_13, K_14, K_15, K_16, K_17, K_18, K_19, K_2, K_20, K_21, K_22, K_23, K_24, K_25, K_26, K_27, K_28, K_29, K_3, K_30, K_31, K_32, K_33, K_34, K_35, K_36, K_37, K_38, K_39, K_4, K_40, K_41, K_42, K_43, K_44, K_45, K_46, K_47, K_48, K_49, K_5, K_50, K_51, K_52, K_53, K_54, K_55, K_56, K_57, K_58, K_59, K_6, K_60, K_61, K_62, K_63, K_64, K_65, K_66, K_67, K_68, K_69, K_7, K_70, K_71, K_72, K_73, K_74, K_75, K_76, K_77, K_78, K_79, K_8, K_80, K_81, K_82, K_83, K_84, K_85, K_86, K_9: symbol MX_Alps_Hybrid:MX-NoLED -> Switch:SW_Push
Connections:
- net col0: now also K_0.2, K_16.2, K_33.2, K_50.2, K_76.2; no longer K_0.1 (COL), K_16.1 (COL), K_33.1 (COL), K_50.1 (COL), K_76.1 (COL)
- net col1: now also K_17.2, K_63.2, K_77.2; no longer K_17.1 (COL), K_63.1 (COL), K_77.1 (COL)
- net col10: now also K_26.2, K_42.2, K_59.2, K_72.2, K_8.2, K_80.2; no longer K_26.1 (COL), K_42.1 (COL), K_59.1 (COL), K_72.1 (COL), K_8.1 (COL), K_80.1 (COL)
- net col11: now also K_27.2, K_43.2, K_60.2, K_73.2, K_81.2, K_9.2; no longer K_27.1 (COL), K_43.1 (COL), K_60.1 (COL), K_73.1 (COL), K_81.1 (COL), K_9.1 (COL)
- net col12: now also K_10.2, K_28.2, K_44.2, K_61.2; no longer K_10.1 (COL), K_28.1 (COL), K_44.1 (COL), K_61.1 (COL)
- net col13: now also K_11.2, K_45.2, K_62.2, K_74.2, K_82.2; no longer K_11.1 (COL), K_45.1 (COL), K_62.1 (COL), K_74.1 (COL), K_82.1 (COL)
- net col14: now also K_12.2, K_29.2, K_46.2, K_83.2; no longer K_12.1 (COL), K_29.1 (COL), K_46.1 (COL), K_83.1 (COL)
- net col15: now also K_13.2, K_30.2, K_47.2, K_84.2; no longer K_13.1 (COL), K_30.1 (COL), K_47.1 (COL), K_84.1 (COL)
- net col16: now also K_14.2, K_31.2, K_48.2, K_75.2, K_85.2; no longer K_14.1 (COL), K_31.1 (COL), K_48.1 (COL), K_75.1 (COL), K_85.1 (COL)
- net col17: now also K_15.2, K_32.2, K_49.2, K_86.2; no longer K_15.1 (COL), K_32.1 (COL), K_49.1 (COL), K_86.1 (COL)
- net col2: now also K_1.2, K_18.2, K_34.2, K_51.2, K_64.2; no longer K_1.1 (COL), K_18.1 (COL), K_34.1 (COL), K_51.1 (COL), K_64.1 (COL)
- net col3: now also K_19.2, K_2.2, K_35.2, K_52.2, K_65.2, K_78.2; no longer K_19.1 (COL), K_2.1 (COL), K_35.1 (COL), K_52.1 (COL), K_65.1 (COL), K_78.1 (COL)
- net col4: now also K_20.2, K_3.2, K_36.2, K_53.2, K_66.2; no longer K_20.1 (COL), K_3.1 (COL), K_36.1 (COL), K_53.1 (COL), K_66.1 (COL)
- net col5: now also K_21.2, K_37.2, K_4.2, K_54.2, K_67.2; no longer K_21.1 (COL), K_37.1 (COL), K_4.1 (COL), K_54.1 (COL), K_67.1 (COL)
- net col6: now also K_22.2, K_38.2, K_55.2, K_68.2, K_79.2; no longer K_22.1 (COL), K_38.1 (COL), K_55.1 (COL), K_68.1 (COL), K_79.1 (COL)
- net col7: now also K_23.2, K_39.2, K_5.2, K_56.2, K_69.2; no longer K_23.1 (COL), K_39.1 (COL), K_5.1 (COL), K_56.1 (COL), K_69.1 (COL)
- net col8: now also K_24.2, K_40.2, K_57.2, K_6.2, K_70.2; no longer K_24.1 (COL), K_40.1 (COL), K_57.1 (COL), K_6.1 (COL), K_70.1 (COL)
- net col9: now also K_25.2, K_41.2, K_58.2, K_7.2, K_71.2; no longer K_25.1 (COL), K_41.1 (COL), K_58.1 (COL), K_7.1 (COL), K_71.1 (COL)
- net at D_34.2 (A): now also K_34.1; no longer K_34.2 (ROW)
- net at D_58.2 (A): now also K_58.1; no longer K_58.2 (ROW)
- net at D_23.2 (A): now also K_23.1; no longer K_23.2 (ROW)
- net at D_78.2 (A): now also K_78.1; no longer K_78.2 (ROW)
- net at D_4.2 (A): now also K_4.1; no longer K_4.2 (ROW)
- net at D_79.2 (A): now also K_79.1; no longer K_79.2 (ROW)
- net at D_84.2 (A): now also K_84.1; no longer K_84.2 (ROW)
- net at D_51.2 (A): now also K_51.1; no longer K_51.2 (ROW)
- net at D_2.2 (A): now also K_2.1; no longer K_2.2 (ROW)
- net at D_82.2 (A): now also K_82.1; no longer K_82.2 (ROW)
- net at D_42.2 (A): now also K_42.1; no longer K_42.2 (ROW)
- net at D_31.2 (A): now also K_31.1; no longer K_31.2 (ROW)
- net at D_35.2 (A): now also K_35.1; no longer K_35.2 (ROW)
- net at D_60.2 (A): now also K_60.1; no longer K_60.2 (ROW)
- net at D_80.2 (A): now also K_80.1; no longer K_80.2 (ROW)
- net at D_33.2 (A): now also K_33.1; no longer K_33.2 (ROW)
- net at D_76.2 (A): now also K_76.1; no longer K_76.2 (ROW)
- net at D_19.2 (A): now also K_19.1; no longer K_19.2 (ROW)
- net at D_86.2 (A): now also K_86.1; no longer K_86.2 (ROW)
- net at D_47.2 (A): now also K_47.1; no longer K_47.2 (ROW)
- net at D_55.2 (A): now also K_55.1; no longer K_55.2 (ROW)
- net at D_28.2 (A): now also K_28.1; no longer K_28.2 (ROW)
- net at D_53.2 (A): now also K_53.1; no longer K_53.2 (ROW)
- net at D_61.2 (A): now also K_61.1; no longer K_61.2 (ROW)
- net at D_63.2 (A): now also K_63.1; no longer K_63.2 (ROW)
- net at D_38.2 (A): now also K_38.1; no longer K_38.2 (ROW)
- net at D_29.2 (A): now also K_29.1; no longer K_29.2 (ROW)
- net at D_3.2 (A): now also K_3.1; no longer K_3.2 (ROW)
- net at D_68.2 (A): now also K_68.1; no longer K_68.2 (ROW)
- net at D_52.2 (A): now also K_52.1; no longer K_52.2 (ROW)
- net at D_44.2 (A): now also K_44.1; no longer K_44.2 (ROW)
- net at D_26.2 (A): now also K_26.1; no longer K_26.2 (ROW)
- net at D_20.2 (A): now also K_20.1; no longer K_20.2 (ROW)
- net at D_37.2 (A): now also K_37.1; no longer K_37.2 (ROW)
- net at D_7.2 (A): now also K_7.1; no longer K_7.2 (ROW)
- net at D_45.2 (A): now also K_45.1; no longer K_45.2 (ROW)
- net at D_17.2 (A): now also K_17.1; no longer K_17.2 (ROW)
- net at D_0.2 (A): now also K_0.1; no longer K_0.2 (ROW)
- net at D_6.2 (A): now also K_6.1; no longer K_6.2 (ROW)
- net at D_1.2 (A): now also K_1.1; no longer K_1.2 (ROW)
- net at D_24.2 (A): now also K_24.1; no longer K_24.2 (ROW)
- net at D_12.2 (A): now also K_12.1; no longer K_12.2 (ROW)
- net at D_77.2 (A): now also K_77.1; no longer K_77.2 (ROW)
- net at D_39.2 (A): now also K_39.1; no longer K_39.2 (ROW)
- net at D_5.2 (A): now also K_5.1; no longer K_5.2 (ROW)
- net at D_16.2 (A): now also K_16.1; no longer K_16.2 (ROW)
- net at D_75.2 (A): now also K_75.1; no longer K_75.2 (ROW)
- net at D_22.2 (A): now also K_22.1; no longer K_22.2 (ROW)
- net at D_64.2 (A): now also K_64.1; no longer K_64.2 (ROW)
- net at D_62.2 (A): now also K_62.1; no longer K_62.2 (ROW)
- net at D_67.2 (A): now also K_67.1; no longer K_67.2 (ROW)
- net at D_73.2 (A): now also K_73.1; no longer K_73.2 (ROW)
- net at D_13.2 (A): now also K_13.1; no longer K_13.2 (ROW)
- net at D_69.2 (A): now also K_69.1; no longer K_69.2 (ROW)
- net at D_14.2 (A): now also K_14.1; no longer K_14.2 (ROW)
- net at D_18.2 (A): now also K_18.1; no longer K_18.2 (ROW)
- net at D_56.2 (A): now also K_56.1; no longer K_56.2 (ROW)
- net at D_66.2 (A): now also K_66.1; no longer K_66.2 (ROW)
- net at D_43.2 (A): now also K_43.1; no longer K_43.2 (ROW)
- net at D_50.2 (A): now also K_50.1; no longer K_50.2 (ROW)
- net at D_49.2 (A): now also K_49.1; no longer K_49.2 (ROW)
- net at D_30.2 (A): now also K_30.1; no longer K_30.2 (ROW)
- net at D_36.2 (A): now also K_36.1; no longer K_36.2 (ROW)
- net at D_72.2 (A): now also K_72.1; no longer K_72.2 (ROW)
- net at D_41.2 (A): now also K_41.1; no longer K_41.2 (ROW)
- net at D_54.2 (A): now also K_54.1; no longer K_54.2 (ROW)
- net at D_85.2 (A): now also K_85.1; no longer K_85.2 (ROW)
- net at D_9.2 (A): now also K_9.1; no longer K_9.2 (ROW)
- net at D_46.2 (A): now also K_46.1; no longer K_46.2 (ROW)
- net at D_10.2 (A): now also K_10.1; no longer K_10.2 (ROW)
- net at D_15.2 (A): now also K_15.1; no longer K_15.2 (ROW)
- net at D_70.2 (A): now also K_70.1; no longer K_70.2 (ROW)
- net at D_74.2 (A): now also K_74.1; no longer K_74.2 (ROW)
- net at D_81.2 (A): now also K_81.1; no longer K_81.2 (ROW)
- net at D_21.2 (A): now also K_21.1; no longer K_21.2 (ROW)
- net at D_25.2 (A): now also K_25.1; no longer K_25.2 (ROW)
- net at D_27.2 (A): now also K_27.1; no longer K_27.2 (ROW)
- net at D_83.2 (A): now also K_83.1; no longer K_83.2 (ROW)
- net at D_57.2 (A): now also K_57.1; no longer K_57.2 (ROW)
- net at D_65.2 (A): now also K_65.1; no longer K_65.2 (ROW)
- net at D_8.2 (A): now also K_8.1; no longer K_8.2 (ROW)
- net at D_40.2 (A): now also K_40.1; no longer K_40.2 (ROW)
- net at D_48.2 (A): now also K_48.1; no longer K_48.2 (ROW)
- net at D_32.2 (A): now also K_32.1; no longer K_32.2 (ROW)
- net at D_59.2 (A): now also K_59.1; no longer K_59.2 (ROW)
- net at D_71.2 (A): now also K_71.1; no longer K_71.2 (ROW)
- net at D_11.2 (A): now also K_11.1; no longer K_11.2 (ROW)
Other:
- moved on the sheet: D_0, D_1, D_10, D_11, D_12, D_13, D_14, D_15, D_16, D_17, D_18, D_19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

Commit message: Removed unused row
Connections:
- net col0: now also Pico0.9 (GPIO6); no longer Pico0.10 (GPIO7)
- net col1: now also Pico0.10 (GPIO7); no longer Pico0.11 (GPIO8)
- net col10: now also Pico0.21 (GPIO16); no longer Pico0.22 (GPIO17)
- net col11: now also Pico0.22 (GPIO17); no longer Pico0.24 (GPIO18)
- net col12: now also Pico0.24 (GPIO18); no longer Pico0.25 (GPIO19)
- net col13: now also Pico0.25 (GPIO19); no longer Pico0.26 (GPIO20)
- net col14: now also Pico0.26 (GPIO20); no longer Pico0.27 (GPIO21)
- net col15: now also Pico0.27 (GPIO21); no longer Pico0.29 (GPIO22)
- net col16: now also Pico0.29 (GPIO22); no longer Pico0.31 (GPIO26_ADC0)
- net col17: now also Pico0.31 (GPIO26_ADC0); no longer Pico0.32 (GPIO27_ADC1)
- net col2: now also Pico0.11 (GPIO8); no longer Pico0.12 (GPIO9)
- net col3: now also Pico0.12 (GPIO9); no longer Pico0.14 (GPIO10)
- net col4: now also Pico0.14 (GPIO10); no longer Pico0.15 (GPIO11)
- net col5: now also Pico0.15 (GPIO11); no longer Pico0.16 (GPIO12)
- net col6: now also Pico0.16 (GPIO12); no longer Pico0.17 (GPIO13)
- net col7: now also Pico0.17 (GPIO13); no longer Pico0.19 (GPIO14)
- net col8: now also Pico0.19 (GPIO14); no longer Pico0.20 (GPIO15)
- net col9: now also Pico0.20 (GPIO15); no longer Pico0.21 (GPIO16)
- net row1: now also D_16.1 (K), D_17.1 (K), D_18.1 (K), D_19.1 (K), D_20.1 (K), D_21.1 (K), D_22.1 (K), D_23.1 (K), D_24.1 (K), D_25.1 (K), D_26.1 (K), D_27.1 (K), D_28.1 (K), D_29.1 (K), D_30.1 (K), D_31.1 (K), D_32.1 (K)
- net row2: now also D_33.1 (K), D_34.1 (K), D_35.1 (K), D_36.1 (K), D_37.1 (K), D_38.1 (K), D_39.1 (K), D_40.1 (K), D_41.1 (K), D_42.1 (K), D_43.1 (K), D_44.1 (K), D_45.1 (K), D_46.1 (K), D_47.1 (K), D_48.1 (K), D_49.1 (K); no longer D_16.1 (K), D_17.1 (K), D_18.1 (K), D_19.1 (K), D_20.1 (K), D_21.1 (K), D_22.1 (K), D_23.1 (K), D_24.1 (K), D_25.1 (K), D_26.1 (K), D_27.1 (K), D_28.1 (K), D_29.1 (K), D_30.1 (K), D_31.1 (K), D_32.1 (K)
- net row3: now also D_50.1 (K), D_51.1 (K), D_52.1 (K), D_53.1 (K), D_54.1 (K), D_55.1 (K), D_56.1 (K), D_57.1 (K), D_58.1 (K), D_59.1 (K), D_60.1 (K), D_61.1 (K), D_62.1 (K); no longer D_33.1 (K), D_34.1 (K), D_35.1 (K), D_36.1 (K), D_37.1 (K), D_38.1 (K), D_39.1 (K), D_40.1 (K), D_41.1 (K), D_42.1 (K), D_43.1 (K), D_44.1 (K), D_45.1 (K), D_46.1 (K), D_47.1 (K), D_48.1 (K), D_49.1 (K)
- net row4: now also D_63.1 (K), D_64.1 (K), D_65.1 (K), D_66.1 (K), D_67.1 (K), D_68.1 (K), D_69.1 (K), D_70.1 (K), D_71.1 (K), D_72.1 (K), D_73.1 (K), D_74.1 (K), D_75.1 (K); no longer D_50.1 (K), D_51.1 (K), D_52.1 (K), D_53.1 (K), D_54.1 (K), D_55.1 (K), D_56.1 (K), D_57.1 (K), D_58.1 (K), D_59.1 (K), D_60.1 (K), D_61.1 (K), D_62.1 (K)
- net row5: now also D_76.1 (K), D_77.1 (K), D_78.1 (K), D_79.1 (K), D_80.1 (K), D_81.1 (K), D_82.1 (K), D_83.1 (K), D_84.1 (K), D_85.1 (K), D_86.1 (K); no longer D_63.1 (K), D_64.1 (K), D_65.1 (K), D_66.1 (K), D_67.1 (K), D_68.1 (K), D_69.1 (K), D_70.1 (K), D_71.1 (K), D_72.1 (K), D_73.1 (K), D_74.1 (K), D_75.1 (K)
- net GND: now reaches Pico0.13 (GND)
- net GND: now also Pico0.18 (GND), Pico0.23 (GND), Pico0.28 (GND), Pico0.3 (GND), Pico0.38 (GND), Pico0.8 (GND)
- removed net row6: D_76.1 (K), D_77.1 (K), D_78.1 (K), D_79.1 (K), D_80.1 (K), D_81.1 (K), D_82.1 (K), D_83.1 (K), D_84.1 (K), D_85.1 (K), D_86.1 (K), Pico0.9 (GPIO6)
Other:
- moved on the sheet: D_0, D_1, D_10, D_11, D_12, D_13, D_14, D_15, D_2, D_3, D_4, D_5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
